File: Filtro.sch (KiCad schematic (older format))
At the start: 12 parts

Commit message: terminando el diseno
Parts:
- renumbered C13 to C10, C14 to C11, C15 to C12, C16 to C13, C7 to C4, C8 to C5, C9 to C6, C10 to C7, C11 to C8, C12 to C9, D1 to D3, D2 to D4
Changed lines of the file:
@@
 Rev "V 0.1.0"
 Comp "PCB PROFESIONAL"
-Comment1 ""
+Comment1 "https://maykolrey.com"
 Comment2 ""
 Comment3 ""
@@
 $EndDescr
 $Comp
-L Device:D_Schottky_x2_ACom_KAK D1
+L Device:D_Schottky_x2_ACom_KAK D3
 U 1 1 5F99AAC6
 P 3600 3550
-F 0 "D1" V 3554 3630 50  0000 L CNN
+F 0 "D3" V 3554 3630 50  0000 L CNN
 F 1 "MBRF1080CTR" V 3450 2750 50  0000 L CNN
 F 2 "Package_TO_SOT_THT:TO-220-3_Vertical" H 3600 3550 50  0001 C CNN
@@
 $EndComp
 $Comp
-L Device:D_Schottky_x2_KCom_AKA D2
+L Device:D_Schottky_x2_KCom_AKA D4
 U 1 1 5F99C051
 P 4200 3550
-F 0 "D2" V 4154 3630 50  0000 L CNN
+F 0 "D4" V 4154 3630 50  0000 L CNN
 F 1 "MBRF1080CT" V 4050 2950 50  0000 L CNN
 F 2 "Package_TO_SOT_THT:TO-220-3_Vertical" H 4200 3550 50  0001 C CNN
@@
 	3600 3150 3900 3150
 $Comp
-L Device:CP1 C7
+L Device:CP1 C4
 U 1 1 5F9A77CF
 P 5900 3350
-F 0 "C7" H 6015 3441 50  0000 L CNN
+F 0 "C4" H 6015 3441 50  0000 L CNN
 F 1 "1000uF" H 6015 3350 50  0000 L CNN
 F 2 "Capacitor_THT:CP_Radial_D10.0mm_P5.00mm" H 5900 3350 50  0001 C CNN
@@
 	3150 3550 3400 3550
 $Comp
-L Device:CP1 C9
+L Device:CP1 C6
 U 1 1 5F9AB366
 P 6450 3350
-F 0 "C9" H 6565 3441 50  0000 L CNN
+F 0 "C6" H 6565 3441 50  0000 L CNN
 F 1 "1000uF" H 6565 3350 50  0000 L CNN
 F 2 "Capacitor_THT:CP_Radial_D10.0mm_P5.00mm" H 6450 3350 50  0001 C CNN
@@
 $EndComp
 $Comp
-L Device:CP1 C11
+L Device:CP1 C8
 U 1 1 5F9ABBD7
 P 7000 3350
-F 0 "C11" H 7115 3441 50  0000 L CNN
+F 0 "C8" H 7115 3441 50  0000 L CNN
 F 1 "1000uF" H 7115 3350 50  0000 L CNN
 F 2 "Capacitor_THT:CP_Radial_D10.0mm_P5.00mm" H 7000 3350 50  0001 C CNN
@@
 $EndComp
 $Comp
-L Device:CP1 C13
+L Device:CP1 C10
 U 1 1 5F9AC26E
 P 7500 3350
-F 0 "C13" H 7615 3441 50  0000 L CNN
+F 0 "C10" H 7615 3441 50  0000 L CNN
 F 1 "1000uF" H 7615 3350 50  0000 L CNN
 F 2 "Capacitor_THT:CP_Radial_D10.0mm_P5.00mm" H 7500 3350 50  0001 C CNN
@@
 $EndComp
 $Comp
-L Device:C C15
+L Device:C C12
 U 1 1 5F9ACB8B
 P 8050 3350
-F 0 "C15" H 8165 3396 50  0000 L CNN
+F 0 "C12" H 8165 3396 50  0000 L CNN
 F 1 "0.1uF" H 8165 3305 50  0000 L CNN
 F 2 "Capacitor_THT:C_Disc_D3.8mm_W2.6mm_P2.50mm" H 8088 3200 50  0001 C CNN
@@
 	7500 3150 7000 3150
 $Comp
-L Device:CP1 C8
+L Device:CP1 C5
 U 1 1 5F9B2E0F
 P 5900 3750
-F 0 "C8" H 6015 3841 50  0000 L CNN
+F 0 "C5" H 6015 3841 50  0000 L CNN
 F 1 "1000uF" H 6015 3750 50  0000 L CNN
 F 2 "Capacitor_THT:CP_Radial_D10.0mm_P5.00mm" H 5900 3750 50  0001 C CNN
@@
 $EndComp
 $Comp
-L Device:CP1 C10
+L Device:CP1 C7
 U 1 1 5F9B2E16
 P 6450 3750
-F 0 "C10" H 6565 3841 50  0000 L CNN
+F 0 "C7" H 6565 3841 50  0000 L CNN
 F 1 "1000uF" H 6565 3750 50  0000 L CNN
 F 2 "Capacitor_THT:CP_Radial_D10.0mm_P5.00mm" H 6450 3750 50  0001 C CNN
@@
 $EndComp
 $Comp
-L Device:CP1 C12
+L Device:CP1 C9
 U 1 1 5F9B2E1D
 P 7000 3750
-F 0 "C12" H 7115 3841 50  0000 L CNN
+F 0 "C9" H 7115 3841 50  0000 L CNN
 F 1 "1000uF" H 7115 3750 50  0000 L CNN
 F 2 "Capacitor_THT:CP_Radial_D10.0mm_P5.00mm" H 7000 3750 50  0001 C CNN
@@
 $EndComp
 $Comp
-L Device:CP1 C14
+L Device:CP1 C11
 U 1 1 5F9B2E24
 P 7500 3750
-F 0 "C14" H 7615 3841 50  0000 L CNN
+F 0 "C11" H 7615 3841 50  0000 L CNN
 F 1 "1000uF" H 7615 3750 50  0000 L CNN
 F 2 "Capacitor_THT:CP_Radial_D10.0mm_P5.00mm" H 7500 3750 50  0001 C CNN
@@
 $EndComp
 $Comp
-L Device:C C16
+L Device:C C13
 U 1 1 5F9B2E2A
 P 8050 3750
-F 0 "C16" H 8165 3796 50  0000 L CNN
+F 0 "C13" H 8165 3796 50  0000 L CNN
 F 1 "0.1uF" H 8165 3705 50  0000 L CNN
 F 2 "Capacitor_THT:C_Disc_D3.8mm_W2.6mm_P2.50mm" H 8088 3600 50  0001 C CNN
@@
 Connection ~ 5900 3550
 $Comp
-L power:GNDREF #PWR021
+L power:GNDREF #PWR024
 U 1 1 5F9BFB4B
 P 8350 3550
-F 0 "#PWR021" H 8350 3300 50  0001 C CNN
+F 0 "#PWR024" H 8350 3300 50  0001 C CNN
 F 1 "GNDREF" V 8355 3422 50  0000 R CNN
 F 2 "" H 8350 3550 50  0001 C CNN
