File: transformacion.sch (KiCad schematic (older format))
At the start: 18 parts, among them Q1 2N3904, Q2 2N3906, Q3 2N3904, Q4 2N3906, Q5 IRFZ44N, Q6 IRFZ44N, Q7 IRFZ44N, Q8 IRFZ44N

Commit message: terminando el diseno
Parts:
- renumbered C6 to C3, R7 to R10, R8 to R11, R9 to R12, R10 to R13, R11 to R14, R12 to R15, R6 to R9
Changed lines of the file:
@@
 Sheet 3 4
 Title "Fuente conmutada +/-36V 250W"
-Date "2020-10-23"
+Date "2020-12-18"
 Rev "V 0.1.0"
 Comp "PCB PROFESIONAL"
-Comment1 ""
+Comment1 "https://maykolrey.com"
 Comment2 ""
 Comment3 ""
@@
 	3300 2350 3300 3050
 $Comp
-L power:+12V #PWR011
+L power:+12V #PWR014
 U 1 1 5F93A361
 P 3750 2000
-F 0 "#PWR011" H 3750 1850 50  0001 C CNN
+F 0 "#PWR014" H 3750 1850 50  0001 C CNN
 F 1 "+12V" H 3765 2173 50  0000 C CNN
 F 2 "" H 3750 2000 50  0001 C CNN
@@
 	3750 2000 3750 2150
 $Comp
-L power:GND #PWR012
+L power:GND #PWR015
 U 1 1 5F93ABB6
 P 3750 3550
-F 0 "#PWR012" H 3750 3300 50  0001 C CNN
+F 0 "#PWR015" H 3750 3300 50  0001 C CNN
 F 1 "GND" H 3755 3377 50  0000 C CNN
 F 2 "" H 3750 3550 50  0001 C CNN
@@
 	3750 3550 3750 3250
 $Comp
-L Device:R R6
+L Device:R R9
 U 1 1 5F93B424
 P 3300 3350
-F 0 "R6" H 3370 3396 50  0000 L CNN
+F 0 "R9" H 3370 3396 50  0000 L CNN
 F 1 "1K" H 3370 3305 50  0000 L CNN
 F 2 "Resistor_THT:R_Axial_DIN0207_L6.3mm_D2.5mm_P10.16mm_Horizontal" V 3230 3350 50  0001 C CNN
@@
 Connection ~ 3300 3050
 $Comp
-L power:GND #PWR09
+L power:GND #PWR012
 U 1 1 5F93BC23
 P 3300 3550
-F 0 "#PWR09" H 3300 3300 50  0001 C CNN
+F 0 "#PWR012" H 3300 3300 50  0001 C CNN
 F 1 "GND" H 3305 3377 50  0000 C CNN
 F 2 "" H 3300 3550 50  0001 C CNN
@@
 	3300 4700 3300 5350
 $Comp
-L power:+12V #PWR013
+L power:+12V #PWR016
 U 1 1 5F93C69A
 P 3750 4350
-F 0 "#PWR013" H 3750 4200 50  0001 C CNN
+F 0 "#PWR016" H 3750 4200 50  0001 C CNN
 F 1 "+12V" H 3765 4523 50  0000 C CNN
 F 2 "" H 3750 4350 50  0001 C CNN
@@
 	3750 4350 3750 4500
 $Comp
-L power:GND #PWR014
+L power:GND #PWR017
 U 1 1 5F93C6A5
 P 3750 5850
-F 0 "#PWR014" H 3750 5600 50  0001 C CNN
+F 0 "#PWR017" H 3750 5600 50  0001 C CNN
 F 1 "GND" H 3755 5677 50  0000 C CNN
 F 2 "" H 3750 5850 50  0001 C CNN
@@
 	3750 5850 3750 5550
 $Comp
-L Device:R R7
+L Device:R R10
 U 1 1 5F93C6B0
 P 3300 5600
-F 0 "R7" H 3370 5646 50  0000 L CNN
+F 0 "R10" H 3370 5646 50  0000 L CNN
 F 1 "1K" H 3370 5555 50  0000 L CNN
 F 2 "Resistor_THT:R_Axial_DIN0207_L6.3mm_D2.5mm_P10.16mm_Horizontal" V 3230 5600 50  0001 C CNN
@@
 Connection ~ 3300 5350
 $Comp
-L power:GND #PWR010
+L power:GND #PWR013
 U 1 1 5F93C6BD
 P 3300 5850
-F 0 "#PWR010" H 3300 5600 50  0001 C CNN
+F 0 "#PWR013" H 3300 5600 50  0001 C CNN
 F 1 "GND" H 3305 5677 50  0000 C CNN
 F 2 "" H 3300 5850 50  0001 C CNN
@@
 Connection ~ 3300 4700
 $Comp
-L Device:R R9
+L Device:R R12
 U 1 1 5F942E7F
 P 4850 2700
-F 0 "R9" V 4643 2700 50  0000 C CNN
+F 0 "R12" V 4643 2700 50  0000 C CNN
 F 1 "10" V 4734 2700 50  0000 C CNN
 F 2 "Resistor_THT:R_Axial_DIN0207_L6.3mm_D2.5mm_P10.16mm_Horizontal" V 4780 2700 50  0001 C CNN
@@
 	5000 2700 5100 2700
 $Comp
-L power:GND #PWR015
+L power:GND #PWR018
 U 1 1 5F944062
 P 5400 3000
-F 0 "#PWR015" H 5400 2750 50  0001 C CNN
+F 0 "#PWR018" H 5400 2750 50  0001 C CNN
 F 1 "GND" H 5405 2827 50  0000 C CNN
 F 2 "" H 5400 3000 50  0001 C CNN
@@
 $EndComp
 $Comp
-L Device:R R8
+L Device:R R11
 U 1 1 5F94627C
 P 4850 1800
-F 0 "R8" V 4643 1800 50  0000 C CNN
+F 0 "R11" V 4643 1800 50  0000 C CNN
 F 1 "10" V 4734 1800 50  0000 C CNN
 F 2 "Resistor_THT:R_Axial_DIN0207_L6.3mm_D2.5mm_P10.16mm_Horizontal" V 4780 1800 50  0001 C CNN
@@
 $EndComp
 $Comp
-L power:GND #PWR017
+L power:GND #PWR020
 U 1 1 5F946283
 P 5900 2100
-F 0 "#PWR017" H 5900 1850 50  0001 C CNN
+F 0 "#PWR020" H 5900 1850 50  0001 C CNN
 F 1 "GND" H 5905 1927 50  0000 C CNN
 F 2 "" H 5900 2100 50  0001 C CNN
@@
 	3750 2700 3750 2850
 $Comp
-L Device:R R10
+L Device:R R13
 U 1 1 5F955E3C
 P 4850 5000
-F 0 "R10" V 4643 5000 50  0000 C CNN
+F 0 "R13" V 4643 5000 50  0000 C CNN
 F 1 "10" V 4734 5000 50  0000 C CNN
 F 2 "Resistor_THT:R_Axial_DIN0207_L6.3mm_D2.5mm_P10.16mm_Horizontal" V 4780 5000 50  0001 C CNN
@@
 	5000 5000 5100 5000
 $Comp
-L power:GND #PWR016
+L power:GND #PWR019
 U 1 1 5F955E43
 P 5400 4650
-F 0 "#PWR016" H 5400 4400 50  0001 C CNN
+F 0 "#PWR019" H 5400 4400 50  0001 C CNN
 F 1 "GND" H 5405 4477 50  0000 C CNN
 F 2 "" H 5400 4650 50  0001 C CNN
@@
 $EndComp
 $Comp
-L Device:R R11
+L Device:R R14
 U 1 1 5F955E50
 P 4850 5800
-F 0 "R11" V 4643 5800 50  0000 C CNN
+F 0 "R14" V 4643 5800 50  0000 C CNN
 F 1 "10" V 4734 5800 50  0000 C CNN
 F 2 "Resistor_THT:R_Axial_DIN0207_L6.3mm_D2.5mm_P10.16mm_Horizontal" V 4780 5800 50  0001 C CNN
@@
 	5000 5800 5600 5800
 $Comp
-L power:GND #PWR018
+L power:GND #PWR021
 U 1 1 5F955E57
 P 5900 5450
-F 0 "#PWR018" H 5900 5200 50  0001 C CNN
+F 0 "#PWR021" H 5900 5200 50  0001 C CNN
 F 1 "GND" H 5905 5277 50  0000 C CNN
 F 2 "" H 5900 5450 50  0001 C CNN
@@
 	3750 5000 3750 5150
 $Comp
-L Transformer:TRANSF5 TR1
+L Transformer:TRANSF5 TR?
 U 1 1 5F95F5B9
 P 7850 3850
-AR Path="/5F95F5B9" Ref="TR1"  Part="1"
+AR Path="/5F95F5B9" Ref="TR?"  Part="1"
 AR Path="/5F9356CE/5F95F5B9" Ref="TR1"  Part="1"
 F 0 "TR1" H 7850 4231 50  0000 C CNN
@@
 	7650 3650 7300 3650
 $Comp
-L power:+12V #PWR019
+L power:+12V #PWR022
 U 1 1 5F9624DF
 P 7100 3800
-F 0 "#PWR019" H 7100 3650 50  0001 C CNN
+F 0 "#PWR022" H 7100 3650 50  0001 C CNN
 F 1 "+12V" H 7115 3973 50  0000 C CNN
 F 2 "" H 7100 3800 50  0001 C CNN
@@
 Connection ~ 5900 6150
 $Comp
-L Device:R R12
+L Device:R R15
 U 1 1 5F97E690
 P 6650 3600
-F 0 "R12" H 6720 3691 50  0000 L CNN
+F 0 "R15" H 6720 3691 50  0000 L CNN
 F 1 "270" H 6720 3600 50  0000 L CNN
 F 2 "Resistor_THT:R_Axial_DIN0309_L9.0mm_D3.2mm_P15.24mm_Horizontal" V 6580 3600 50  0001 C CNN
@@
 $EndComp
 $Comp
-L Device:C C6
+L Device:C C3
 U 1 1 5F97EBB7
 P 6650 4100
-F 0 "C6" H 6765 4146 50  0000 L CNN
+F 0 "C3" H 6765 4146 50  0000 L CNN
 F 1 "0.33uF" H 6765 4055 50  0000 L CNN
 F 2 "Capacitor_THT:C_Disc_D4.3mm_W1.9mm_P5.00mm" H 6688 3950 50  0001 C CNN
@@
 	8250 4050 8050 4050
 $Comp
-L power:GNDREF #PWR020
+L power:GNDREF #PWR023
 U 1 1 5F99D4E4
 P 8300 3850
-F 0 "#PWR020" H 8300 3600 50  0001 C CNN
+F 0 "#PWR023" H 8300 3600 50  0001 C CNN
 F 1 "GNDREF" V 8305 3722 50  0000 R CNN
 F 2 "" H 8300 3850 50  0001 C CNN

Commit message: separando el modulo de oscilacion en otra  placa
Parts:
- removed F1: Fuse, Fuse:Fuse_Blade_ATO_directSolder, symbol Device:Fuse
- removed Q1, Q3: 2N3904, Package_TO_SOT_THT:TO-92L_Inline, symbol Device:Q_NPN_EBC
- removed Q2, Q4: 2N3906, Package_TO_SOT_THT:TO-92L_Inline, symbol Device:Q_PNP_EBC
- removed R10, R9: 1K, Resistor_THT:R_Axial_DIN0207_L6.3mm_D2.5mm_P10.16mm_Horizontal, symbol Device:R
Connections:
- net +12V: now also TR1.2
- net In_A: now also R11.2, R12.2
- net In_B: now also R13.2, R14.2
Changed lines of the file:
@@
 Comment4 ""
 $EndDescr
-$Comp
-L Device:Q_PNP_EBC Q2
-U 1 1 5F935993
-P 3650 3050
-F 0 "Q2" H 3840 3004 50  0000 L CNN
-F 1 "2N3906" H 3840 3095 50  0000 L CNN
-F 2 "Package_TO_SOT_THT:TO-92L_Inline" H 3850 3150 50  0001 C CNN
-F 3 "~" H 3650 3050 50  0001 C CNN
-	1    3650 3050
-	1    0    0    1
-$EndComp
-$Comp
-L Device:Q_NPN_EBC Q1
-U 1 1 5F937A97
-P 3650 2350
-F 0 "Q1" H 3840 2396 50  0000 L CNN
-F 1 "2N3904" H 3840 2305 50  0000 L CNN
-F 2 "Package_TO_SOT_THT:TO-92L_Inline" H 3850 2450 50  0001 C CNN
-F 3 "~" H 3650 2350 50  0001 C CNN
-	1    3650 2350
-	1    0    0    -1
-$EndComp
-Wire Wire Line
-	3750 2550 3750 2700
-Wire Wire Line
-	3450 2350 3300 2350
-Wire Wire Line
-	3300 2350 3300 3050
-$Comp
-L power:+12V #PWR014
-U 1 1 5F93A361
-P 3750 2000
-F 0 "#PWR014" H 3750 1850 50  0001 C CNN
-F 1 "+12V" H 3765 2173 50  0000 C CNN
-F 2 "" H 3750 2000 50  0001 C CNN
-F 3 "" H 3750 2000 50  0001 C CNN
-	1    3750 2000
-	1    0    0    -1
-$EndComp
-Wire Wire Line
-	3750 2000 3750 2150
-$Comp
-L power:GND #PWR015
-U 1 1 5F93ABB6
-P 3750 3550
-F 0 "#PWR015" H 3750 3300 50  0001 C CNN
-F 1 "GND" H 3755 3377 50  0000 C CNN
-F 2 "" H 3750 3550 50  0001 C CNN
-F 3 "" H 3750 3550 50  0001 C CNN
-	1    3750 3550
-	1    0    0    -1
-$EndComp
-Wire Wire Line
-	3750 3550 3750 3250
-$Comp
-L Device:R R9
-U 1 1 5F93B424
-P 3300 3350
-F 0 "R9" H 3370 3396 50  0000 L CNN
-F 1 "1K" H 3370 3305 50  0000 L CNN
-F 2 "Resistor_THT:R_Axial_DIN0207_L6.3mm_D2.5mm_P10.16mm_Horizontal" V 3230 3350 50  0001 C CNN
-F 3 "~" H 3300 3350 50  0001 C CNN
-	1    3300 3350
-	1    0    0    -1
-$EndComp
-Wire Wire Line
-	3300 3050 3450 3050
-Wire Wire Line
-	3300 3200 3300 3050
-Connection ~ 3300 3050
-$Comp
-L power:GND #PWR012
-U 1 1 5F93BC23
-P 3300 3550
-F 0 "#PWR012" H 3300 3300 50  0001 C CNN
-F 1 "GND" H 3305 3377 50  0000 C CNN
-F 2 "" H 3300 3550 50  0001 C CNN
-F 3 "" H 3300 3550 50  0001 C CNN
-	1    3300 3550
-	1    0    0    -1
-$EndComp
-Wire Wire Line
-	3300 3550 3300 3500
-Text HLabel 3100 2350 0    50   Input ~ 0
-In_A
-Wire Wire Line
-	3100 2350 3300 2350
-Connection ~ 3300 2350
-$Comp
-L Device:Q_PNP_EBC Q4
-U 1 1 5F93C683
-P 3650 5350
-F 0 "Q4" H 3840 5304 50  0000 L CNN
-F 1 "2N3906" H 3840 5395 50  0000 L CNN
-F 2 "Package_TO_SOT_THT:TO-92L_Inline" H 3850 5450 50  0001 C CNN
-F 3 "~" H 3650 5350 50  0001 C CNN
-	1    3650 5350
-	1    0    0    1
-$EndComp
-$Comp
-L Device:Q_NPN_EBC Q3
-U 1 1 5F93C68D
-P 3650 4700
-F 0 "Q3" H 3840 4746 50  0000 L CNN
-F 1 "2N3904" H 3840 4655 50  0000 L CNN
-F 2 "Package_TO_SOT_THT:TO-92L_Inline" H 3850 4800 50  0001 C CNN
-F 3 "~" H 3650 4700 50  0001 C CNN
-	1    3650 4700
-	1    0    0    -1
-$EndComp
-Wire Wire Line
-	3750 4900 3750 5000
-Wire Wire Line
-	3450 4700 3300 4700
-Wire Wire Line
-	3300 4700 3300 5350
-$Comp
-L power:+12V #PWR016
-U 1 1 5F93C69A
-P 3750 4350
-F 0 "#PWR016" H 3750 4200 50  0001 C CNN
-F 1 "+12V" H 3765 4523 50  0000 C CNN
-F 2 "" H 3750 4350 50  0001 C CNN
-F 3 "" H 3750 4350 50  0001 C CNN
-	1    3750 4350
-	1    0    0    -1
-$EndComp
-Wire Wire Line
-	3750 4350 3750 4500
-$Comp
-L power:GND #PWR017
-U 1 1 5F93C6A5
-P 3750 5850
-F 0 "#PWR017" H 3750 5600 50  0001 C CNN
-F 1 "GND" H 3755 5677 50  0000 C CNN
-F 2 "" H 3750 5850 50  0001 C CNN
-F 3 "" H 3750 5850 50  0001 C CNN
-	1    3750 5850
-	1    0    0    -1
-$EndComp
-Wire Wire Line
-	3750 5850 3750 5550
-$Comp
-L Device:R R10
-U 1 1 5F93C6B0
-P 3300 5600
-F 0 "R10" H 3370 5646 50  0000 L CNN
-F 1 "1K" H 3370 5555 50  0000 L CNN
-F 2 "Resistor_THT:R_Axial_DIN0207_L6.3mm_D2.5mm_P10.16mm_Horizontal" V 3230 5600 50  0001 C CNN
-F 3 "~" H 3300 5600 50  0001 C CNN
-	1    3300 5600
-	1    0    0    -1
-$EndComp
-Wire Wire Line
-	3300 5350 3450 5350
-Wire Wire Line
-	3300 5450 3300 5350
-Connection ~ 3300 5350
-$Comp
-L power:GND #PWR013
-U 1 1 5F93C6BD
-P 3300 5850
-F 0 "#PWR013" H 3300 5600 50  0001 C CNN
-F 1 "GND" H 3305 5677 50  0000 C CNN
-F 2 "" H 3300 5850 50  0001 C CNN
-F 3 "" H 3300 5850 50  0001 C CNN
-	1    3300 5850
-	1    0    0    -1
-$EndComp
-Wire Wire Line
-	3300 5850 3300 5750
-Text HLabel 3100 4700 0    50   Input ~ 0
+Text HLabel 4400 5000 0    50   Input ~ 0
 In_B
-Wire Wire Line
-	3100 4700 3300 4700
-Connection ~ 3300 4700
 $Comp
 L Device:R R12
@@
 Wire Wire Line
 	5900 2100 5900 2000
-Connection ~ 3750 2700
-Wire Wire Line
-	3750 2700 3750 2850
 $Comp
 L Device:R R13
@@
 	4550 5000 4700 5000
 Wire Wire Line
-	4550 5000 3750 5000
-Connection ~ 4550 5000
-Wire Wire Line
 	4700 5800 4550 5800
 Wire Wire Line
 	4550 5000 4550 5800
-Connection ~ 3750 5000
-Wire Wire Line
-	3750 5000 3750 5150
 $Comp
 L Transformer:TRANSF5 TR?
@@
 	1    0    0    -1
 $EndComp
-$Comp
-L Device:Fuse F1
-U 1 1 5F963652
-P 7400 3850
-F 0 "F1" V 7203 3850 50  0000 C CNN
-F 1 "Fuse" V 7294 3850 50  0000 C CNN
-F 2 "Fuse:Fuse_Blade_ATO_directSolder" V 7330 3850 50  0001 C CNN
-F 3 "~" H 7400 3850 50  0001 C CNN
-	1    7400 3850
-	0    1    1    0
-$EndComp
-Wire Wire Line
-	7550 3850 7650 3850
-Wire Wire Line
-	7250 3850 7100 3850
 Wire Wire Line
 	7100 3850 7100 3800
 Wire Wire Line
-	3750 2700 4550 2700
-Wire Wire Line
 	4700 1800 4550 1800
 Wire Wire Line
 	4550 1800 4550 2700
-Connection ~ 4550 2700
 Wire Wire Line
 	4550 2700 4700 2700
@@
 	1    0    0    1
 $EndComp
+Wire Wire Line
+	4400 5000 4550 5000
+Connection ~ 4550 5000
+Text HLabel 4350 2700 0    50   Input ~ 0
+In_A
+Wire Wire Line
+	4350 2700 4550 2700
+Connection ~ 4550 2700
+Wire Wire Line
+	7100 3850 7650 3850
 $EndSCHEMATC
